File: wired-sculpt.kicad_pcb (KiCad board)
At the start: 2 copper layers, 40 x 50 mm, 39 parts, among them J1 10103594-0001LF, J2 FFC3B07-30-T, J3 AVR-ISP-6 - NOT FITTED, Q1 BSS84AK,215, Q2 2N7002BK, SW1 FSMSM, SW2 S2B-PH-K-S(LF)(SN), U1 USBLC6-2SC6, U2 LM2776DBVT, U3 AT90USB1286-AU, Y1 TSX-3225 16.0000MF18X-AC0

Commit message: modified for fabrication and assembly by JLCPCB
Parts:
- removed C12: CL10B104KB8NNNC, Capacitor_SMD:C_0603_1608Metric
- removed the J3 at (134.8, 76.4)
- removed Q1: BSS84AK,215, Package_TO_SOT_SMD:SOT-23
- removed Q2: 2N7002BK, Package_TO_SOT_SMD:SOT-23
- removed R10, R9: ERJ-3GEYJ331V, Resistor_SMD:R_0603_1608Metric
- removed R11: ERJ-PA3J560V, Resistor_SMD:R_0603_1608Metric
- removed R12, R7: ERJ-PA3F22R0V, Resistor_SMD:R_0603_1608Metric
- removed R8: ERJ-PA3J472V, Resistor_SMD:R_0603_1608Metric
- removed SW2: S2B-PH-K-S(LF)(SN), Connector_JST:JST_PH_S2B-PH-K_1x02_P2.00mm_Horizontal
- removed U3: AT90USB1286-AU, Package_QFP:TQFP-64_14x14mm_P0.8mm
- added D2: Red, LED_SMD:LED_0603_1608Metric_Castellated, F.Cu at (150.8, 47.7)
- added J2: AVR-ISP-6 - NOT FITTED, Connector_IDC:IDC-Header_2x03_P2.54mm_Horizontal, B.Cu at (153.7, 44.8)
- C1: value CL21A475KOFNNNE -> 100n; footprint Capacitor_SMD:C_0805_2012Metric -> Capacitor_SMD:C_0603_1608Metric
- C10, C11: value CL10B104KB8NNNC -> 22u
- C2: value CL21B104KACNNNC -> 10u; footprint Capacitor_SMD:C_0805_2012Metric -> Capacitor_SMD:C_0603_1608Metric
- C3: value CL21B103KBANNNC -> 12p; footprint Capacitor_SMD:C_0805_2012Metric -> Capacitor_SMD:C_0603_1608Metric
- C4: value CL10A105KA8NNNC -> 12p
- C5: value CL10A105KA8NNNC -> 1u
- C6: value CL10A105KA8NNNC -> 100n
- C7, C8: value 06035A160JAT2A -> 100n
- C9: value CL10A105KA8NNNC -> 22u
- D1: value 150080GS75000 -> BAV99; footprint LED_SMD:LED_0603_1608Metric_Castellated -> Package_TO_SOT_SMD:SOT-23
- J1: footprint Connector_USB:USB_Micro-B_Amphenol_10103594-0001LF_Horizontal -> Connector_USB:USB_Micro-B_Molex-105017-0001
- R1: value ERJ-PA3F22R0V -> 100
- R2: value ERJ-PA3F22R0V -> 22; footprint Resistor_SMD:R_0603_1608Metric -> Resistor_SMD:R_0402_1005Metric
- R3: value ERJ-PA3J472V -> 22; footprint Resistor_SMD:R_0603_1608Metric -> Resistor_SMD:R_0402_1005Metric
- R4: value ERJ-3EKF8873V -> 470k
- R5: value ERJ-PA3J473V -> 680
- R6: value ERJ-3GEYJ331V -> 680
- SW1: value FSMSM -> MJTP1117; footprint Button_Switch_SMD:SW_SPST_FSMSM -> kmj_custom:SW_Tactile_SPST_Angled_MJTP1117
- U1: value USBLC6-2SC6 -> SRV05-4-P-T7
- U2: value LM2776DBVT -> AT90USB1286-AU; footprint Package_TO_SOT_SMD:SOT-23-6 -> Package_QFP:TQFP-64_14x14mm_P0.8mm
- Y1: value TSX-3225 16.0000MF18X-AC0 -> 16M
- moved SW1 34.4 mm to (157.1, 70.9)
- moved R1 34.2 mm to (131.4, 39.7), turned to 0 degrees
- moved C3 28.8 mm to (137.9, 43.7), turned to 90 degrees
- moved C4 25.4 mm to (140.8, 41.2), turned to 180 degrees
- moved C7 25.2 mm to (146.2, 64.7)
- moved R6 20.3 mm to (131.4, 41.3), turned to 0 degrees
- moved R5 20.2 mm to (150.8, 49.2)
- moved C11 18.2 mm to (148.8, 44.0), turned to 270 degrees
- moved J1 17.7 mm to (157.3, 57.3)
- moved U2 16.7 mm to (140.2, 54.4), turned to 180 degrees
- moved R3 16.3 mm to (150.0, 58.1), turned to 0 degrees
- moved C1 14.8 mm to (136.6, 64.7), turned to 90 degrees
- moved U1 14.4 mm to (152.9, 57.6), turned to 270 degrees
- moved C2 13.1 mm to (152.9, 61.1), turned to 90 degrees
- moved C9 11.5 mm to (147.3, 44.0)
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- renumbered J2 to J3
Connections:
- C10 pad 2: VBUS -> Net-(C10-Pad2)
- C11 pad 1: GND -> Net-(C11-Pad1)
- C11 pad 2: VBUS -> Net-(C11-Pad2)
- C3 pad 1: GND -> Net-(C3-Pad1)
- C3 pad 2: VBUS -> GND
- C4 pad 2: Net-(C4-Pad2) -> GND
- C5 pad 1: GND -> Net-(C5-Pad1)
- C5 pad 2: VBUS -> GND
- C6 pad 2: -5V -> VBUS
- C7 pad 1: Net-(C7-Pad1) -> GND
- C7 pad 2: GND -> VBUS
- C8 pad 1: Net-(C8-Pad1) -> GND
- C8 pad 2: GND -> VBUS
- C9 pad 1: Net-(C9-Pad1) -> Net-(C11-Pad1)
- C9 pad 2: GND -> Net-(C11-Pad2)
- D1 pad 1: GND -> Net-(C10-Pad2)
- D1 pad 2: Net-(D1-Pad2) -> GND
- J1 pad 2: /Din- -> /D-
- J1 pad 3: /Din+ -> /D+
- J3 pad 10: PE1 -> /COL_12
- J3 pad 11: Net-(J2-Pad11) -> /COL_11
- J3 pad 12: Net-(J2-Pad12) -> /COL_10
- J3 pad 13: Net-(J2-Pad13) -> /COL_9
- J3 pad 14: Net-(J2-Pad14) -> /COL_8
- J3 pad 15: Net-(J2-Pad15) -> /COL_7
- J3 pad 16: Net-(J2-Pad16) -> /COL_6
- J3 pad 17: Net-(J2-Pad17) -> /COL_5
- J3 pad 18: Net-(J2-Pad18) -> /COL_4
- J3 pad 19: Net-(J2-Pad19) -> /COL_3
- J3 pad 2: Net-(J2-Pad2) -> /GREEN_K
- J3 pad 20: Net-(J2-Pad20) -> /COL_2
- J3 pad 21: Net-(J2-Pad21) -> /COL_1
- J3 pad 22: Net-(J2-Pad22) -> /ROW_8
- J3 pad 23: Net-(J2-Pad23) -> /ROW_7
- J3 pad 24: Net-(J2-Pad24) -> /ROW_6
- J3 pad 25: Net-(J2-Pad25) -> /ROW_5
- J3 pad 26: Net-(J2-Pad26) -> /ROW_4
- J3 pad 27: PF7 -> /ROW_3
- J3 pad 28: PF6 -> /ROW_2
- J3 pad 29: PF5 -> /ROW_1
- J3 pad 3: Net-(J2-Pad3) -> /RED_A
- J3 pad 30: PF4 -> /FN_SW
- J3 pad 4: Net-(J2-Pad4) -> /COL_18
- J3 pad 5: Net-(J2-Pad5) -> /COL_17
- J3 pad 6: Net-(J2-Pad6) -> /COL_16
- J3 pad 7: Net-(J2-Pad7) -> /COL_15
- J3 pad 8: Net-(J2-Pad8) -> /COL_14
- J3 pad 9: PE0 -> /COL_13
- R1 pad 1: /D+ -> /GREEN_K
- R1 pad 2: /Dout+ -> Net-(C10-Pad2)
- R2 pad 1: /D- -> /DZ+
- R2 pad 2: /Dout- -> /D+
- R3 pad 1: Net-(R3-Pad1) -> /DZ-
- R3 pad 2: GND -> /D-
- R4 pad 2: PF4 -> /FN_SW
- R5 pad 1: Net-(Q1-Pad1) -> Net-(D2-Pad2)
- R5 pad 2: VBUS -> LED
- R6 pad 1: Net-(Q1-Pad1) -> /RED_A
- R6 pad 2: GREEN+ -> Net-(R6-Pad2)
- SW1 pad 2: Net-(R10-Pad2) -> RST
- U1 pad 1: /Din- -> /D+
- U1 pad 3: /Din+ -> Net-(U1-Pad3)
- U1 pad 4: /Dout+ -> Net-(U1-Pad4)
- U1 pad 6: /Dout- -> /D-
- U2 pad 1: -5V -> Net-(U2-Pad1)
- U2 pad 2: GND -> Net-(U2-Pad2)
- U2 pad 4: PB0 -> /DZ-
- U2 pad 5: Net-(C4-Pad1) -> /DZ+
- U2 pad 6: Net-(C4-Pad2) -> GND
- Y1 pad 1: Net-(C7-Pad1) -> Net-(C3-Pad1)
- Y1 pad 3: Net-(C8-Pad1) -> Net-(C4-Pad1)
Routing:
- net VBUS: track 138.6 -> 14.3 mm
- net RST: track 48.3 -> 123.9 mm, vias 3 -> 0
- net -5V: track 40.5 -> 0.00 mm, vias 2 -> 0
- net RED+: track 40.1 -> 0.00 mm, vias 2 -> 0
- net GND: track 62.8 -> 32.6 mm, vias 13 -> 16
- net Net-(R10-Pad2): track 27.9 -> 0.00 mm
- net MISO: track 37.0 -> 10.5 mm, vias 2 -> 0
- net Net-(R6-Pad2): track 0.00 -> 25.1 mm
- net PF4: track 24.0 -> 0.00 mm
- net /FN_SW: track 0.00 -> 23.0 mm
- net /ROW_1: track 0.00 -> 22.4 mm
- net PF5: track 19.9 -> 0.00 mm
- net PF6: track 19.1 -> 0.00 mm
- net Net-(J2-Pad2): track 18.5 -> 0.00 mm
- net MOSI: track 33.1 -> 14.7 mm, vias 2 -> 0
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- added copper zone on F.Cu, net VBUS
Other:
- net class Default: clearance 0.2 -> 0.127; trace_width 0.25 -> 0.127; via_dia 0.7 -> 0.6; via_drill 0.4 -> 0.3
- net class Fat removed
- rule pad_to_mask_clearance: 0.0508 -> 0
- rule trace_clearance: 0.2 -> 0.127
- rule trace_min: 0.2 -> 0.127
- board text added: "Wired Sculpt KMJ_mod github.com/chadaustin/wired-sculpt-pcb 2021-05-17"
- board text removed: "Wired Sculpt 0.4 Chad Austin 2021-05-08"
