File: wired-sculpt.sch (KiCad schematic (older format))
At the start: 39 parts, among them J1 10103594-0001LF, J2 FFC3B07-30-T, J3 AVR-ISP-6 - NOT FITTED, Q1 BSS84AK,215, Q2 2N7002BK, SW1 FSMSM, SW2 S2B-PH-K-S(LF)(SN), U1 USBLC6-2SC6, U2 LM2776DBVT, U3 AT90USB1286-AU, Y1 TSX-3225 16.0000MF18X-AC0

Commit message: modified for fabrication and assembly by JLCPCB
Parts:
- removed C12: CL10B104KB8NNNC, Capacitor_SMD:C_0603_1608Metric, symbol Device:C
- removed C3: CL21B103KBANNNC, Capacitor_SMD:C_0805_2012Metric, symbol Device:C
- removed Q1: BSS84AK,215, Package_TO_SOT_SMD:SOT-23, symbol Transistor_FET:BSS84
- removed Q2: 2N7002BK, Package_TO_SOT_SMD:SOT-23, symbol Transistor_FET:2N7002
- removed R10, R9: ERJ-3GEYJ331V, Resistor_SMD:R_0603_1608Metric, symbol Device:R_US
- removed R11: ERJ-PA3J560V, Resistor_SMD:R_0603_1608Metric, symbol Device:R_US
- removed R12, R7: ERJ-PA3F22R0V, Resistor_SMD:R_0603_1608Metric, symbol Device:R_US
- removed R3, R8: ERJ-PA3J472V, Resistor_SMD:R_0603_1608Metric, symbol Device:R_US
- removed SW2: S2B-PH-K-S(LF)(SN), Connector_JST:JST_PH_S2B-PH-K_1x02_P2.00mm_Horizontal, symbol Connector:Conn_01x02_Female
- removed U2: LM2776DBVT, Package_TO_SOT_SMD:SOT-23-6, symbol Regulator_SwitchedCapacitor:LM2776
- added C7: 100n, Capacitor_SMD:C_0603_1608Metric, symbol Device:C
- added D1: BAV99, Package_TO_SOT_SMD:SOT-23, symbol Diode:BAV99
- added R1: 100, Resistor_SMD:R_0603_1608Metric, symbol Device:R_US
- C1: value CL21A475KOFNNNE -> 100n; footprint Capacitor_SMD:C_0805_2012Metric -> Capacitor_SMD:C_0603_1608Metric; Desc (none) -> 100nF ±10% 50V X7R 0603; LCSC (none) -> C14663; Mfr (none) -> YAGEO; Mfr_part (none) -> CC0603KRX7R9BB104
- C10, C11: value CL10B104KB8NNNC -> 22u; Desc (none) -> 22uF ±20% 6.3V X5R 0603; LCSC (none) -> C59461; Mfr (none) -> Samsung Electro-Mechanics; Mfr_part (none) -> CL10A226MQ8NRNC
- C2: value CL21B104KACNNNC -> 10u; footprint Capacitor_SMD:C_0805_2012Metric -> Capacitor_SMD:C_0603_1608Metric; Desc (none) -> 10uF ±10% 10V X5R; LCSC (none) -> C19702; Mfr (none) -> Samsung Electro-Mechanics; Mfr_part (none) -> CL10A106KP8NNNC
- C3: renamed from C7; value CL10C160JB8NNNC -> 12p; Desc (none) -> 12pF ±5% 50V C0G 0603; LCSC (none) -> C38523; Mfr (none) -> Samsung Electro-Mechanics; Mfr_part (none) -> CL10C120JB8NNNC
- C4: value CL10A105KA8NNNC -> 12p; Desc (none) -> 12pF ±5% 50V C0G 0603; LCSC (none) -> C38523; Mfr (none) -> Samsung Electro-Mechanics; Mfr_part (none) -> CL10C120JB8NNNC
- C5: value CL10A105KA8NNNC -> 1u; Desc (none) -> 1uF ±10% 50V X5R 0603; LCSC (none) -> C15849; Mfr (none) -> Samsung Electro-Mechanics; Mfr_part (none) -> CL10A105KB8NNNC
- C6: value CL10A105KA8NNNC -> 100n; Desc (none) -> 100nF ±10% 50V X7R 0603; LCSC (none) -> C14663; Mfr (none) -> YAGEO; Mfr_part (none) -> CC0603KRX7R9BB104
- C8: value CL10C160JB8NNNC -> 100n; Desc (none) -> 100nF ±10% 50V X7R 0603; LCSC (none) -> C14663; Mfr (none) -> YAGEO; Mfr_part (none) -> CC0603KRX7R9BB104
- C9: value CL10A105KA8NNNC -> 22u; Desc (none) -> 22uF ±20% 6.3V X5R 0603; LCSC (none) -> C59461; Mfr (none) -> Samsung Electro-Mechanics; Mfr_part (none) -> CL10A226MQ8NRNC
- D2: renamed from D1; value 150080GS75000 -> Red; Desc (none) -> Light Emitting Diodes (LED) Red 520~625nm 90~100mcd@20mA To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; LCSC (none) -> C2286; Mfr (none) -> Hubei KENTO Elec; Mfr_part (none) -> KT-0603R
- J1: footprint Connector_USB:USB_Micro-B_Amphenol_10103594-0001LF_Horizontal -> Connector_USB:USB_Micro-B_Molex-105017-0001
- J2: renamed from J3; footprint Connector_IDC:IDC-Header_2x03_P2.54mm_Vertical -> Connector_IDC:IDC-Header_2x03_P2.54mm_Horizontal
- R2: renamed from R1; value ERJ-PA3F22R0V -> 22; footprint Resistor_SMD:R_0603_1608Metric -> Resistor_SMD:R_0402_1005Metric; Desc (none) -> 22Ω ±1% 1/16W ±200ppm/℃ 0402; LCSC (none) -> C25092; Mfr (none) -> UNI-ROYAL(Uniroyal Elec); Mfr_part (none) -> 0402WGF220JTCE
- R3: renamed from R2; value ERJ-PA3F22R0V -> 22; footprint Resistor_SMD:R_0603_1608Metric -> Resistor_SMD:R_0402_1005Metric; Desc (none) -> 22Ω ±1% 1/16W ±200ppm/℃ 0402; LCSC (none) -> C25092; Mfr (none) -> UNI-ROYAL(Uniroyal Elec); Mfr_part (none) -> 0402WGF220JTCE
- R4: value ERJ-3EKF8873V -> 470k; Desc (none) -> 470kΩ ±1% 0.1W ±100ppm/℃ 0603; LCSC (none) -> C23178; Mfr (none) -> UNI-ROYAL(Uniroyal Elec); Mfr_part (none) -> 0603WAF4703T5E
- R5: value ERJ-PA3J473V -> 680; Desc (none) -> 680Ω ±1% 0.1W ±100ppm/℃ 0603; LCSC (none) -> C23228; Mfr (none) -> UNI-ROYAL(Uniroyal Elec); Mfr_part (none) -> 0603WAF6800T5E
- R6: value ERJ-3GEYJ331V -> 680; Desc (none) -> 680Ω ±1% 0.1W ±100ppm/℃ 0603; LCSC (none) -> C23228; Mfr (none) -> UNI-ROYAL(Uniroyal Elec); Mfr_part (none) -> 0603WAF6800T5E
- SW1: value FSMSM -> MJTP1117; footprint Button_Switch_SMD:SW_SPST_FSMSM -> kmj_custom:SW_Tactile_SPST_Angled_MJTP1117; Desc (none) -> SWITCH TACTILE SPST-NO 0.05A 12V; Mfr (none) -> APEM Inc; Mfr_part (none) -> MJTP1117
- U1: value USBLC6-2SC6 -> SRV05-4-P-T7; symbol Power_Protection:USBLC6-2SC6 -> Power_Protection:SRV05-4; Desc (none) -> TVS SOT-23-6; LCSC (none) -> C85364; Mfr (none) -> ProTek Devices; Mfr_part (none) -> SRV05-4-P-T7
- U2: renamed from U3; Desc (none) -> TQFP-64 MCU; LCSC (none) -> C619147; Mfr (none) -> Microchip Tech; Mfr_part (none) -> AT90USB1286-AU
- Y1: value TSX-3225 16.0000MF18X-AC0 -> 16M; Desc (none) -> SMD Crystal Resonators 16MHz ±10ppm SMD-3225_4P; LCSC (none) -> C13738; Mfr (none) -> Yangxing Tech; Mfr_part (none) -> X322516MLB4SI
- renumbered J2 to J3
Connections:
- net labels added: COL_1, COL_10, COL_11, COL_12, COL_13, COL_14, COL_15, COL_16, COL_17, COL_18, COL_2, COL_3, COL_4, COL_5, COL_6, COL_7, COL_8, COL_9, DZ+, DZ-, FN_SW, GREEN_K, RED_A, ROW_1, ROW_2, ROW_3, ROW_4, ROW_5, ROW_6, ROW_7, ROW_8
- net labels removed: -5V, Din+, Din-, Dout+, Dout-, GREEN+, GREEN-, PB0, PE0, PE1, PF4, PF5, PF6, PF7, RED+
- wire segments 151 -> 133
- no-connect marks 15 -> 18
Other:
- note added: "Toggle this line to \nprovide inverted \nvoltage to green led"
- moved on the sheet: C3, D2, H1, H2, H3, J1, J2, J3, R2, R3, R4, SW1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
